Commit message: added franka, new scenes, problemsets, done cleanup in scenes

File: data/scenes/industrial/industrial.urdf (robot description, URDF)
Before this commit: robot industrial, 1 links, 0 joints
Links:
- removed link bookshelf
- added link industrial_env, mass 0; collision mesh filename=industrial.obj; visual mesh filename=industrial.obj

Commit message: fixed industrial env

File: data/scenes/industrial/industrial.urdf (robot description, URDF)
Before this commit: robot industrial, 1 links, 0 joints
Links:
- removed link industrial_env
- added link bookshelf, mass 0; collision mesh filename=industrial-acd.obj; visual mesh filename=industrial-acd.obj
