Commit message: fixed urdf + changed sphere placement code to work ONLY for UR10

File: data/robots/ur10/ur10.urdf (robot description, URDF)
Before this commit: robot ur10, 9 links, 8 joints
Links:
- link forearm_link: geometry collision mesh filename=package://meshes/ur10/collision/Forearm.dae; visual mesh filename=package://meshes/ur10/visual/Forearm.dae
- link upper_arm_link: geometry collision mesh filename=package://meshes/ur10/collision/UpperArm.dae; visual mesh filename=package://meshes/ur10/visual/UpperArm.dae
- link wrist_1_link: geometry collision mesh filename=package://meshes/ur10/collision/Wrist1.dae; visual mesh filename=package://meshes/ur10/visual/Wrist1.dae

File: data/robots/wam/wam.urdf (robot description, URDF)
Before this commit: robot wam, 10 links, 9 joints
Joints:
- joint wam/wam_fixed_joint: origin xyz=0.0 0.0 1.0 rpy=0 0 0 -> xyz=0.0 0.0 0.0 rpy=0 0 0
