Commit message: WAM robot working / changed URDF for it / changed offset and FK code for it

File: data/robots/wam/wam.urdf (robot description, URDF)
Before this commit: robot wam, 10 links, 9 joints
Links:
- link wam/base_link: geometry collision mesh filename=package://sw_meshes/base_link_convex.dae; visual mesh filename=package://sw_meshes/base_link_fine.stl
- link wam/forearm_link: geometry collision mesh filename=package://sw_meshes/elbow_link_convex.dae; collision mesh filename=package://sw_meshes/forearm_link_convex_decomposition.dae
- link wam/shoulder_pitch_link: geometry collision mesh filename=package://sw_meshes/shoulder_pitch_link_convex.dae; visual mesh filename=package://sw_meshes/shoulder_pitch_link_fine.stl
- link wam/shoulder_yaw_link: geometry collision mesh filename=package://sw_meshes/shoulder_link_convex_decomposition.dae; visual mesh filename=package://sw_meshes/shoulder_link_fine.stl
- link wam/upper_arm_link: geometry collision mesh filename=package://sw_meshes/upper_arm_link_convex_decomposition.dae; visual mesh filename=package://sw_meshes/upper_arm_link_fine.stl
- link wam/wrist_palm_stump_link: geometry visual sphere radius=0.0575
- link wam/wrist_pitch_link: geometry collision mesh filename=package://sw_meshes/wrist_pitch_link_convex_decomposition.d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; visual mesh filename=package://sw_meshes/wrist_pitch_link_fine.stl
- link wam/wrist_yaw_link: geometry collision mesh filename=package://sw_meshes/wrist_yaw_link_convex_decomposition.dae; visual mesh filename=package://sw_meshes/wrist_yaw_link_fine.stl

Commit message: added WAM hand and spheres

File: data/robots/wam/wam.urdf (robot description, URDF)
Before this commit: robot wam, 10 links, 9 joints
Links:
- added link wam/bhand/bhand_grasp_link, mass 0.000001
- added link wam/bhand/bhand_palm_link, mass 0.50573; collision mesh filename=package://sw_meshes/bhand/bhand_palm_link_convex_decomposit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; visual mesh filename=package://sw_meshes/bhand/bhand_palm_fine.stl
- added link wam/bhand/bhand_palm_surface_link, mass 0.000001
- added link wam/bhand/finger_1/dist_link, mass 0.041377; collision mesh filename=package://sw_meshes/bhand/bhand_finger_dist_link_convex.dae; visual mesh filename=package://sw_meshes/bhand/bhand_finger_dist_link_fine.stl
- added link wam/bhand/finger_1/med_link, mass 0.062139; collision mesh filename=package://sw_meshes/bhand/bhand_finger_med_link_convex.dae; visual mesh filename=package://sw_meshes/bhand/bhand_finger_med_link_fine.stl
- added link wam/bhand/finger_1/prox_link, mass 0.14109; collision mesh filename=package://sw_meshes/bhand/bhand_finger_prox_link_convex_dec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; visual mesh filename=package://sw_meshes/bhand/bhand_finger_prox_link_fine.stl
- added link wam/bhand/finger_1/tip_link, mass 1E-6
- added link wam/bhand/finger_2/dist_link, mass 0.041377; collision mesh filename=package://sw_meshes/bhand/bhand_finger_dist_link_convex.dae; visual mesh filename=package://sw_meshes/bhand/bhand_finger_dist_link_fine.stl
- added link wam/bhand/finger_2/med_link, mass 0.062139; collision mesh filename=package://sw_meshes/bhand/bhand_finger_med_link_convex.dae; visual mesh filename=package://sw_meshes/bhand/bhand_finger_med_link_fine.stl
- added link wam/bhand/finger_2/prox_link, mass 0.14109; collision mesh filename=package://sw_meshes/bhand/bhand_finger_prox_link_convex_dec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; visual mesh filename=package://sw_meshes/bhand/bhand_finger_prox_link_fine.stl
- added link wam/bhand/finger_2/tip_link, mass 1E-6
- added link wam/bhand/finger_3/dist_link, mass 0.041377; collision mesh filename=package://sw_meshes/bhand/bhand_finger_dist_link_convex.dae; visual mesh filename=package://sw_meshes/bhand/bhand_finger_dist_link_fine.stl
- added link wam/bhand/finger_3/med_link, mass 0.062139; collision mesh filename=package://sw_meshes/bhand/bhand_finger_med_link_convex.dae; visual mesh filename=package://sw_meshes/bhand/bhand_finger_med_link_fine.stl
- added link wam/bhand/finger_3/tip_link, mass 1E-6
- link wam/wrist_palm_stump_link: geometry visual sphere radius=0.024; visual sphere radius=0.024
Joints:
- added joint wam/bhand/bhand_base_joint: type fixed, parent wam/wrist_palm_link, child wam/bhand/bhand_palm_link, origin xyz=0 0 0.06 rpy=0 0 0
- added joint wam/bhand/bhand_grasp_joint: type fixed, parent wam/bhand/bhand_palm_link, child wam/bhand/bhand_grasp_link, origin xyz=0 0 0.12 rpy=0 0 0, limit lower=0 upper=3.141592653589793 effort=5 velocity=5.0
- added joint wam/bhand/bhand_palm_surface_joint: type fixed, parent wam/bhand/bhand_palm_link, child wam/bhand/bhand_palm_surface_link, origin xyz=0 0 0.08 rpy=0 0 0, limit lower=0 upper=3.141592653589793 effort=5 velocity=5.0
- added joint wam/bhand/finger_1/dist_joint: type revolute, parent wam/bhand/finger_1/med_link, child wam/bhand/finger_1/dist_link, origin xyz=0.06994 0.003 0.0 rpy=0 0 0.7853981633974483, axis 0 0 1, limit lower=0 upper=0.8377580409572781 effort=5 velocity=5.00
- added joint wam/bhand/finger_1/med_joint: type revolute, parent wam/bhand/finger_1/prox_link, child wam/bhand/finger_1/med_link, origin xyz=0.05 0.0 0.03390 rpy=1.5707963267948966 0 0, axis 0 0 1, limit lower=0 upper=2.443460952792061 effort=5 velocity=5.00
- added joint wam/bhand/finger_1/prox_joint: type revolute, parent wam/bhand/bhand_palm_link, child wam/bhand/finger_1/prox_link, origin xyz=-0.025 0.0 0.0415 rpy=0 0 -1.5707963267948966, axis 0 0 -1, limit lower=0 upper=3.141592653589793 effort=5 velocity=5.0
- added joint wam/bhand/finger_1/tip_joint: type fixed, parent wam/bhand/finger_1/dist_link, child wam/bhand/finger_1/tip_link, origin xyz=0.05 0.0 0.0 rpy=0 0 0
- added joint wam/bhand/finger_2/dist_joint: type revolute, parent wam/bhand/finger_2/med_link, child wam/bhand/finger_2/dist_link, origin xyz=0.06994 0.003 0.0 rpy=0 0 0.7853981633974483, axis 0 0 1, limit lower=0 upper=0.8377580409572781 effort=5 velocity=5.00
- added joint wam/bhand/finger_2/med_joint: type revolute, parent wam/bhand/finger_2/prox_link, child wam/bhand/finger_2/med_link, origin xyz=0.05 0.0 0.03390 rpy=1.5707963267948966 0 0, axis 0 0 1, limit lower=0 upper=2.443460952792061 effort=5 velocity=5.00
- added joint wam/bhand/finger_2/prox_joint: type revolute, parent wam/bhand/bhand_palm_link, child wam/bhand/finger_2/prox_link, origin xyz=0.025 0.0 0.0415 rpy=0 0 -1.5707963267948966, axis 0 0 1, limit lower=0 upper=3.141592653589793 effort=5 velocity=5.0
- added joint wam/bhand/finger_2/tip_joint: type fixed, parent wam/bhand/finger_2/dist_link, child wam/bhand/finger_2/tip_link, origin xyz=0.05 0.0 0.0 rpy=0 0 0
- added joint wam/bhand/finger_3/dist_joint: type revolute, parent wam/bhand/finger_3/med_link, child wam/bhand/finger_3/dist_link, origin xyz=0.06994 0.003 0.0 rpy=0 0 0.7853981633974483, axis 0 0 1, limit lower=0 upper=0.8377580409572781 effort=5 velocity=5.00
- added joint wam/bhand/finger_3/med_joint: type revolute, parent wam/bhand/bhand_palm_link, child wam/bhand/finger_3/med_link, origin xyz=0 0.05 0.0754 rpy=1.5707963267948966 0 1.5707963267948966, axis 0 0 1, limit lower=0 upper=2.443460952792061 effort=5 velocity=5.00
- added joint wam/bhand/finger_3/tip_joint: type fixed, parent wam/bhand/finger_3/dist_link, child wam/bhand/finger_3/tip_link, origin xyz=0.05 0.0 0.0 rpy=0 0 0

Commit message: testing out some things for WAM

File: data/robots/wam/wam.urdf (robot description, URDF)
Before this commit: robot wam, 24 links, 23 joints
Links:
- link wam/forearm_link: geometry collision mesh filename=package://sw_meshes/elbow_link_convex.dae; collision mesh filename=package://sw_meshes/forearm_link_convex_decomposition.dae
- link wam/shoulder_pitch_link: geometry collision mesh filename=package://sw_meshes/shoulder_pitch_link_convex.dae; visual mesh filename=package://sw_meshes/shoulder_pitch_link_fine.stl

Commit message: fix some states for benchmark, make spheres on wam bigger

File: data/robots/wam/wam.urdf (robot description, URDF)
Before this commit: robot wam, 24 links, 23 joints
Links:
- link wam/forearm_link: geometry collision mesh filename=package://sw_meshes/elbow_link_convex.dae; collision mesh filename=package://sw_meshes/forearm_link_convex_decomposition.dae
- link wam/shoulder_pitch_link: geometry collision mesh filename=package://sw_meshes/shoulder_pitch_link_convex.dae; visual mesh filename=package://sw_meshes/shoulder_pitch_link_fine.stl
- link wam/wrist_palm_stump_link: geometry visual sphere radius=0.034; visual sphere radius=0.034
- link wam/wrist_pitch_link: geometry collision mesh filename=package://sw_meshes/wrist_pitch_link_convex_decomposition.d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; visual mesh filename=package://sw_meshes/wrist_pitch_link_fine.stl
