Commit message: removed spheres from robot, opened gripper to show grasp position better

File: data/robots/franka/franka_spheres.urdf (robot description, URDF)
Before this commit: robot panda, 12 links, 11 joints
Links:
- link panda_link0: geometry collision mesh filename=package://franka/meshes/collision/link0.stl scale=1.0 1.0 1.0; visual mesh filename=package://franka/meshes/visual/link0.dae scale=1.0 1.0 1.0
- link panda_link1: geometry collision mesh filename=package://franka/meshes/collision/link1.stl scale=1.0 1.0 1.0; visual mesh filename=package://franka/meshes/visual/link1.dae scale=1.0 1.0 1.0
- link panda_link2: geometry collision mesh filename=package://franka/meshes/collision/link2.stl scale=1.0 1.0 1.0; visual mesh filename=package://franka/meshes/visual/link2.dae scale=1.0 1.0 1.0
- link panda_link3: geometry collision mesh filename=package://franka/meshes/collision/link3.stl scale=1.0 1.0 1.0; visual mesh filename=package://franka/meshes/visual/link3.dae scale=1.0 1.0 1.0
- link panda_link4: geometry collision mesh filename=package://franka/meshes/collision/link4.stl scale=1.0 1.0 1.0; visual mesh filename=package://franka/meshes/visual/link4.dae scale=1.0 1.0 1.0
- link panda_link5: geometry collision mesh filename=package://franka/meshes/collision/link5.stl scale=1.0 1.0 1.0; visual mesh filename=package://franka/meshes/visual/link5.dae scale=1.0 1.0 1.0
- link panda_link6: geometry collision mesh filename=package://franka/meshes/collision/link6.stl scale=1.0 1.0 1.0; visual mesh filename=package://franka/meshes/visual/link6.dae scale=1.0 1.0 1.0
- link panda_link7: geometry collision mesh filename=package://franka/meshes/collision/link7.stl scale=1.0 1.0 1.0; visual mesh filename=package://franka/meshes/visual/link7.dae scale=1.0 1.0 1.0

Commit message: new grasping experiment, fixed franka EE alignment

File: data/robots/franka/franka_spheres.urdf (robot description, URDF)
Before this commit: robot panda, 12 links, 11 joints
Joints:
- joint panda_hand_joint: origin xyz=0.0 0.0 0.0 rpy=2.8683722064215544e-12 6.924822375381442e-12 0.0 -> xyz=0.0 0.0 0.0 rpy=0 0 0.0
- joint panda_joint8: origin xyz=0.0 4.845297921863539e-28 0.10700000000000003 rpy=0.0 -0.0 0.0 -> xyz=0.0 4.845297921863539e-28 0.10700000000000003 rpy=0.0 -0.0 -0.7874
